Commit message: moveit assistant not load

File: ur5/Universal_Robots_ROS2_Description-jazzy/urdf/ur_macro.xacro (robot description, xacro)
@@ -1,5 +1,5 @@
 <?xml version="1.0"?>
 <robot xmlns:xacro="http://wiki.ros.org/xacro">
-<xacro:include filename="$(find robotiq_2f_85_gripper_visualization)/urdf/robotiq_arg2f_85_model_macro.xacro"/>
+<!-- <xacro:include filename="$(find robotiq_2f_85_gripper_visualization)/urdf/robotiq_arg2f_85_model_macro.xacro"/> -->
   <!--
     Base UR robot series xacro macro.
@@ -384,9 +384,6 @@
       <child link="${tf_prefix}tool0"/>
     </joint>
-    <xacro:include filename="$(find robotiq_2f_85_gripper_visualization)/urdf/robotiq_arg2f_85_model_macro.xacro"/>
-    <!-- Include the gripper Xacro file  -->
+    <!-- <xacro:include filename="$(find robotiq_2f_85_gripper_visualization)/urdf/robotiq_arg2f_85_model_macro.xacro"/>
     <xacro:robotiq_arg2f_85 prefix=""/>
-    <!-- Attach the gripper to tool0 -->
-    <!-- Attach gripper to wrist_3_link with corrected rotation -->
     <joint name="${tf_prefix}gripper_joint" type="fixed">
       <parent link="${tf_prefix}tool0"/>
@@ -396,6 +393,5 @@
         <disableFixedJointLumping>true</disableFixedJointLumping>
       </gazebo>
-    </joint>
-    <!-- Define the gripper with a meaningful prefix -->
+    </joint>  -->
   </xacro:macro>
 </robot>

File: ur5/Universal_Robots_ROS2_GZ_Simulation/ur_simulation_gz/urdf/ur_gz.urdf.xacro (robot description, xacro)
@@ -1,4 +1,4 @@
 <?xml version="1.0"?>
-<robot xmlns:xacro="http://wiki.ros.org/xacro" name="$(arg name)">
+<robot xmlns:xacro="http://wiki.ros.org/xacro" name="ur">
   <!-- robot name parameter -->
   <xacro:arg name="name" default="ur"/>
@@ -8,5 +8,5 @@
   <!-- possible 'ur_type' values: ur3, ur3e, ur5, ur5e, ur7e, ur10, ur10e, ur12e, ur16e, ur15, ur20, ur30 -->
   <!-- the default value should raise an error in case this was called without defining the type -->
-  <xacro:arg name="ur_type" default="ur5x"/>
+  <xacro:arg name="ur_type" default="ur5e"/>
   <!-- parameters -->
   <xacro:arg name="tf_prefix" default="" />
